File: KiCad/KeeBar_BottomPlate/KeeBar_BottomPlate.kicad_pcb (KiCad board)
At the start: 2 copper layers, 376 x 86.5 mm, 10 parts, among them M2_1 Val**, M2_2 Val**, M2_3 Val**, M2_4 Val**, M2_5 Val**, M2_6 Val**, M2_7 Val**, M2_8 Val**, M2_9 Val**

Commit message: v1.1設計の更新
Parts:
- M2_1, M2_2, M2_3, M2_4, M2_5, M2_6, M2_7, M2_8, M2_9: footprint kbd_Hole:m2_Screw_Hole_EdgeCuts -> kbd_Hole:m2_Screw_Hole
- moved M2_3 25.0 mm to (287.0, 62.0)
- moved M2_8 23.7 mm to (287.0, 104.8)
- moved M2_4 16.2 mm to (361.5, 62.0)
- moved M2_9 12.2 mm to (361.5, 104.8)
- moved M2_5 5.83 mm to (205.0, 83.5)
- moved M2_7 3.34 mm to (117.0, 104.8)
- moved M2_1 2.50 mm to (50.0, 62.0)
- moved M2_2 2.50 mm to (117.0, 62.0)
- moved M2_6 2.30 mm to (50.0, 104.8)
- renumbered G*** to ?
Other:
- outline, holes or cut-outs redrawn
- board text added: "KeeBar v1.1 @ymkn"
- board text removed: "KeeBar Bottom Plate v1.0 @ymkn"
