File: KiCad/KeeBar_PCB/KeeBar.kicad_sch (KiCad schematic)
At the start: 121 parts, among them SW1 SW_Push, SW10 SW_Push, SW11 SW_Push, SW12 SW_Push, SW13 SW_Push, SW14 SW_Push, SW15 SW_Push, SW16 SW_Push, SW17 SW_Push, SW18 SW_Push, SW19 SW_Push, SW2 SW_Push, SW20 SW_Push, SW21 SW_Push, SW22 SW_Push, SW23 SW_Push, SW24 SW_Push, SW25 SW_Push, SW26 SW_Push, SW27 SW_Push, SW28 SW_Push, SW29 SW_Push, SW3 SW_Push, SW30 SW_Push, SW31 SW_Push, SW32 SW_Push, SW33 SW_Push, SW34 SW_Push, SW35 SW_Push, SW36 SW_Push, SW37 SW_Push, SW38 SW_Push, SW39 SW_Push, SW4 SW_Push, SW40 SW_Push, SW41 SW_Push, SW42 SW_Push, SW43 SW_Push, SW44 SW_Push, SW45 SW_Push, SW46 SW_Push, SW47 SW_Push, SW48 SW_Push, SW49 SW_Push, SW5 SW_Push, SW50 SW_Push, SW51 SW_Push, SW52 SW_Push, SW53 SW_Push, SW54 SW_Push, SW55 SW_Push, SW56 SW_Push, SW57 SW_Push, SW58 SW_Push, SW59 SW_Push, SW6 SW_Push, SW60 SW_Push, SW7 SW_Push, SW8 SW_Push, SW9 SW_Push, U1 rp2040-zero

Commit message: v1.1設計の更新
Parts:
- added SW15-2: SW_Push, PCM_Switch_Keyboard_Hotswap_Kailh:SW_Hotswap_Kailh_MX_1.50u, symbol Switch:SW_Push
- added SW16-2: SW_Push, PCM_Switch_Keyboard_Hotswap_Kailh:SW_Hotswap_Kailh_MX_1.00u, symbol Switch:SW_Push
- added SW53-2: SW_Push, PCM_Switch_Keyboard_Hotswap_Kailh:SW_Hotswap_Kailh_MX_2.00u, symbol Switch:SW_Push
- SW1, SW48: footprint MX_Only:MXOnly-1.5U-Hotswap -> PCM_Switch_Keyboard_Hotswap_Kailh:SW_Hotswap_Kailh_MX_1.50u; JLCPCB Part # (none) -> C5156480
- SW10, SW11, SW12, SW13, SW14, SW18, SW19, SW2, SW20, SW21, SW22, SW23, SW24, SW25, SW26, SW27, SW28, SW29, SW3, SW30, SW33, SW34, SW35, SW36, SW37, SW38, SW39, SW4, SW40, SW41, SW42, SW43, SW44, SW45, SW47, SW49, SW5, SW58, SW59, SW6, SW60, SW7, SW8, SW9: footprint MX_Only:MXOnly-1U-Hotswap -> PCM_Switch_Keyboard_Hotswap_Kailh:SW_Hotswap_Kailh_MX_1.00u; JLCPCB Part # (none) -> C5156480
- SW15: footprint MX_Only:MXOnly-1.5U-Hotswap -> PCM_Switch_Keyboard_Hotswap_Kailh:SW_Hotswap_Kailh_MX_1.00u; JLCPCB Part # (none) -> C5156480
- SW16: footprint MX_Only:MXOnly-1U-Hotswap -> PCM_Switch_Keyboard_Hotswap_Kailh:SW_Hotswap_Kailh_MX_1.50u; JLCPCB Part # (none) -> C5156480
- SW17: footprint MX_Only:MXOnly-1.75U-Hotswap -> PCM_Switch_Keyboard_Hotswap_Kailh:SW_Hotswap_Kailh_MX_1.75u; JLCPCB Part # (none) -> C5156480
- SW31: footprint MX_Only:MXOnly-2.25U-Hotswap -> PCM_Switch_Keyboard_Hotswap_Kailh:SW_Hotswap_Kailh_MX_2.25u; JLCPCB Part # (none) -> C5156480
- SW32: footprint MX_Only:MXOnly-2U-Hotswap -> PCM_Switch_Keyboard_Hotswap_Kailh:SW_Hotswap_Kailh_MX_2.00u; JLCPCB Part # (none) -> C5156480
- SW46, SW50, SW51, SW55, SW56, SW57: footprint MX_Only:MXOnly-1.25U-Hotswap -> PCM_Switch_Keyboard_Hotswap_Kailh:SW_Hotswap_Kailh_MX_1.25u; JLCPCB Part # (none) -> C5156480
- SW52: footprint MX_Only:MXOnly-2.75U-Hotswap -> PCM_Switch_Keyboard_Hotswap_Kailh:SW_Hotswap_Kailh_MX_2.75u; JLCPCB Part # (none) -> C5156480
- SW53: footprint MX_Only:MXOnly-1.5U-Hotswap -> PCM_Switch_Keyboard_Hotswap_Kailh:SW_Hotswap_Kailh_MX_7.00u; JLCPCB Part # (none) -> C5156480
- SW54: footprint MX_Only:MXOnly-2.75U-Hotswap -> PCM_Switch_Keyboard_Hotswap_Kailh:SW_Hotswap_Kailh_MX_2.25u; JLCPCB Part # (none) -> C5156480
Connections:
- net COL14: now also SW15-2.1
- net COL15: now also SW16-2.1
- net COL7: now also SW53-2.1
- net at D16.2 (A), SW16.2: now also SW16-2.2
- net at D15.2 (A), SW15.2: now also SW15-2.2
- net at D53.2 (A), SW53.2: now also SW53-2.2
Other:
- moved on the sheet: D53
