File: KiCad/KeeBar_PCB/KeeBar.kicad_pcb (KiCad board)
At the start: 2 copper layers, 376 x 86.5 mm, 141 parts, among them M2_1 Val**, M2_2 Val**, M2_3 Val**, M2_4 Val**, M2_5 Val**, M2_6 Val**, M2_7 Val**, M2_8 Val**, M2_9 Val**, SW1 SW_Push, SW10 SW_Push, SW11 SW_Push, SW12 SW_Push, SW13 SW_Push, SW14 SW_Push, SW15 SW_Push, SW16 SW_Push, SW17 SW_Push, SW18 SW_Push, SW19 SW_Push, SW2 SW_Push, SW20 SW_Push, SW21 SW_Push, SW22 SW_Push, SW23 SW_Push, SW24 SW_Push, SW25 SW_Push, SW26 SW_Push, SW27 SW_Push, SW28 SW_Push, SW29 SW_Push, SW3 SW_Push, SW30 SW_Push, SW31 SW_Push, SW32 SW_Push, SW33 SW_Push, SW34 SW_Push, SW35 SW_Push, SW36 SW_Push, SW37 SW_Push, SW38 SW_Push, SW39 SW_Push, SW4 SW_Push, SW40 SW_Push, SW41 SW_Push, SW42 SW_Push, SW43 SW_Push, SW44 SW_Push, SW45 SW_Push, SW46 SW_Push, SW47 SW_Push, SW48 SW_Push, SW49 SW_Push, SW5 SW_Push, SW50 SW_Push, SW51 SW_Push, SW52 SW_Push, SW53 SW_Push, SW54 SW_Push, SW55 SW_Push, SW56 SW_Push, SW57 SW_Push, SW58 SW_Push, SW59 SW_Push, SW6 SW_Push, SW60 SW_Push, SW7 SW_Push, SW8 SW_Push, SW9 SW_Push, U1 rp2040-zero

Commit message: v1.1設計の更新
Parts:
- removed REF**: Stabilizer_Cherry_MX_7.00u, Mounting_Keyboard_Stabilizer:Stabilizer_Cherry_MX_7.00u
- removed REF** (x3): Stabilizer_Cherry_MX_2.00u, Mounting_Keyboard_Stabilizer:Stabilizer_Cherry_MX_2.00u
- removed REF** (x3): Stabilizer_Cherry_MX_3.00u, Mounting_Keyboard_Stabilizer:Stabilizer_Cherry_MX_3.00u
- removed REF**: Stabilizer_Cherry_MX_6.25u, Mounting_Keyboard_Stabilizer:Stabilizer_Cherry_MX_6.25u
- added ?: Stabilizer_Cherry_MX_2.00u, PCM_Mounting_Keyboard_Stabilizer:Stabilizer_Cherry_MX_2.00u, F.Cu at (235.7, 114.3)
- added ?: Stabilizer_Cherry_MX_6.25u, PCM_Mounting_Keyboard_Stabilizer:Stabilizer_Cherry_MX_6.25u, F.Cu at (190.5, 114.3)
- added ?: Stabilizer_Cherry_MX_7.00u, PCM_Mounting_Keyboard_Stabilizer:Stabilizer_Cherry_MX_7.00u, F.Cu at (190.5, 114.3)
- added ?: Stabilizer_Cherry_MX_2.00u, PCM_Mounting_Keyboard_Stabilizer:Stabilizer_Cherry_MX_2.00u, F.Cu at (195.3, 114.3)
- added ?: Stabilizer_Cherry_MX_2.00u, PCM_Mounting_Keyboard_Stabilizer:Stabilizer_Cherry_MX_2.00u, F.Cu at (150.0, 114.3)
- added SW15-2: SW_Push, PCM_Switch_Keyboard_Hotswap_Kailh:SW_Hotswap_Kailh_MX_1.50u, F.Cu at (333.4, 52.4)
- added SW16-2: SW_Push, PCM_Switch_Keyboard_Hotswap_Kailh:SW_Hotswap_Kailh_MX_1.00u, F.Cu at (357.2, 52.4)
- added SW53-2: SW_Push, PCM_Switch_Keyboard_Hotswap_Kailh:SW_Hotswap_Kailh_MX_2.00u, F.Cu at (195.3, 114.3)
- ? (x2): renamed from REF**; footprint Mounting_Keyboard_Stabilizer:Stabilizer_Cherry_MX_2.00u -> PCM_Mounting_Keyboard_Stabilizer:Stabilizer_Cherry_MX_2.00u
- SW1, SW48: footprint Switch_Keyboard_Hotswap_Kailh:SW_Hotswap_Kailh_MX_1.50u -> PCM_Switch_Keyboard_Hotswap_Kailh:SW_Hotswap_Kailh_MX_1.50u
- SW10, SW11, SW12, SW13, SW14, SW18, SW19, SW2, SW20, SW21, SW22, SW23, SW24, SW25, SW26, SW27, SW28, SW29, SW3, SW30, SW33, SW34, SW35, SW36, SW37, SW38, SW39, SW4, SW40, SW41, SW42, SW43, SW44, SW45, SW47, SW49, SW5, SW58, SW59, SW6, SW60, SW7, SW8, SW9: footprint Switch_Keyboard_Hotswap_Kailh:SW_Hotswap_Kailh_MX_1.00u -> PCM_Switch_Keyboard_Hotswap_Kailh:SW_Hotswap_Kailh_MX_1.00u
- SW15: footprint Switch_Keyboard_Hotswap_Kailh:SW_Hotswap_Kailh_MX_1.50u -> PCM_Switch_Keyboard_Hotswap_Kailh:SW_Hotswap_Kailh_MX_1.00u
- SW16: footprint Switch_Keyboard_Hotswap_Kailh:SW_Hotswap_Kailh_MX_1.00u -> PCM_Switch_Keyboard_Hotswap_Kailh:SW_Hotswap_Kailh_MX_1.50u
- SW17: footprint Switch_Keyboard_Hotswap_Kailh:SW_Hotswap_Kailh_MX_1.75u -> PCM_Switch_Keyboard_Hotswap_Kailh:SW_Hotswap_Kailh_MX_1.75u
- SW31: footprint Switch_Keyboard_Hotswap_Kailh:SW_Hotswap_Kailh_MX_2.25u -> PCM_Switch_Keyboard_Hotswap_Kailh:SW_Hotswap_Kailh_MX_2.25u
- SW32: footprint Switch_Keyboard_Hotswap_Kailh:SW_Hotswap_Kailh_MX_2.00u -> PCM_Switch_Keyboard_Hotswap_Kailh:SW_Hotswap_Kailh_MX_2.00u
- SW46, SW50, SW51, SW55, SW56, SW57: footprint Switch_Keyboard_Hotswap_Kailh:SW_Hotswap_Kailh_MX_1.25u -> PCM_Switch_Keyboard_Hotswap_Kailh:SW_Hotswap_Kailh_MX_1.25u
- SW52: footprint Switch_Keyboard_Hotswap_Kailh:SW_Hotswap_Kailh_MX_2.75u -> PCM_Switch_Keyboard_Hotswap_Kailh:SW_Hotswap_Kailh_MX_2.75u
- SW53: footprint Switch_Keyboard_Hotswap_Kailh:SW_Hotswap_Kailh_MX_1.50u -> PCM_Switch_Keyboard_Hotswap_Kailh:SW_Hotswap_Kailh_MX_7.00u
- SW54: footprint Switch_Keyboard_Hotswap_Kailh:SW_Hotswap_Kailh_MX_2.75u -> PCM_Switch_Keyboard_Hotswap_Kailh:SW_Hotswap_Kailh_MX_2.25u
- moved M2_3 25.0 mm to (287.0, 62.0)
- moved M2_8 23.7 mm to (287.0, 104.8)
- moved M2_4 16.2 mm to (361.5, 62.0)
- moved M2_9 12.2 mm to (361.5, 104.8)
- moved D53 12.0 mm to (178.6, 119.1)
- moved D54 11.9 mm to (235.7, 109.5)
- moved D52 11.0 mm to (150.0, 109.5)
- moved M2_5 5.83 mm to (205.0, 83.5)
- moved D15 5.35 mm to (338.2, 60.9)
- moved D16 5.32 mm to (352.4, 60.9)
- moved SW54 4.76 mm to (235.7, 114.3), turned to 180 degrees
- moved SW15 4.76 mm to (328.6, 52.4)
- moved SW16 4.76 mm to (352.4, 52.4)
- moved M2_7 3.34 mm to (117.0, 104.8)
- moved M2_1 2.50 mm to (50.0, 62.0)
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- renumbered G*** to ?
Routing:
- net ROW3: track 465.3 -> 543.9 mm
- net Net-(D53-A): track 13.0 -> 48.4 mm, vias 0 -> 2
- net COL8: track 341.1 -> 376.3 mm
- net COL7: track 292.9 -> 326.8 mm
- net Net-(D15-A): track 13.0 -> 42.0 mm
- net COL10: track 282.3 -> 308.1 mm
- net Net-(D16-A): track 13.0 -> 36.6 mm
- net COL9: track 306.0 -> 329.3 mm
- net COL14: track 180.3 -> 202.8 mm, vias 0 -> 2
- net ROW0: track 398.1 -> 408.8 mm
- net COL13: track 191.0 -> 200.8 mm
- net Net-(D59-A): track 12.0 -> 19.4 mm
- net GND: track 7.47 -> 0.17 mm, vias 23 -> 24
- net COL6: track 327.6 -> 322.4 mm
- net COL11: track 251.8 -> 256.2 mm
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Other:
- outline, holes or cut-outs redrawn
- board text added: "(1.5u)"
- board text added: "(1u)"
- board text added: "(single)"
- board text added: "(split)"
- board text added: "2u"
- board text added: "2u/7u"
- board text added: "6.25u"
- board text added: "7u"
- board text added: "KeeBar v1.1 @ymkn"
- board text added: "M2"
- board text removed: "KeeBar v1.0 @ymkn"

Commit message: 1.1発注断面
Routing:
- net COL15: track 145.1 -> 145.5 mm, vias 4 -> 5
Changed lines of the file:
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@@
   (via (at 340 125) (size 0.8) (drill 0.4) (layers "F.Cu" "B.Cu") (free) (net 80))
   (via (at 180 125) (size 0.8) (drill 0.4) (layers "F.Cu" "B.Cu") (free) (net 80))
+  (segment (start 360.4 71.8) (end 360.4 69) (width 0.25) (layer "F.Cu") (net 82))
   (segment (start 368.95 82.313604) (end 368.95 76.45) (width 0.25) (layer "F.Cu") (net 82))
   (segment (start 369.6 75.8) (end 369.8 75.8) (width 0.25) (layer "F.Cu") (net 82))
-  (segment (start 364.9 58) (end 364.9 67) (width 0.25) (layer "F.Cu") (net 82))
   (segment (start 375 106) (end 375 88.363604) (width 0.25) (layer "F.Cu") (net 82))
+  (segment (start 360.4 69) (end 364.9 64.5) (width 0.25) (layer "F.Cu") (net 82))
+  (segment (start 364.9 64.5) (end 364.9 58) (width 0.25) (layer "F.Cu") (net 82))
   (segment (start 375 88.363604) (end 368.95 82.313604) (width 0.25) (layer "F.Cu") (net 82))
   (segment (start 368.95 76.45) (end 369.6 75.8) (width 0.25) (layer "F.Cu") (net 82))
   (segment (start 378.6775 109.6775) (end 375 106) (width 0.25) (layer "F.Cu") (net 82))
   (via (at 378.6775 109.6775) (size 0.8) (drill 0.4) (layers "F.Cu" "B.Cu") (net 82))
-  (via (at 364.9 67) (size 0.8) (drill 0.4) (layers "F.Cu" "B.Cu") (net 82))
+  (via (at 360.4 71.8) (size 0.8) (drill 0.4) (layers "F.Cu" "B.Cu") (net 82))
+  (via (at 360.4 68.9) (size 0.8) (drill 0.4) (layers "F.Cu" "B.Cu") (net 82))
   (via (at 364.9 58) (size 0.8) (drill 0.4) (layers "F.Cu" "B.Cu") (net 82))
   (via (at 369.8 75.8) (size 0.8) (drill 0.4) (layers "F.Cu" "B.Cu") (net 82))
   (segment (start 376.545228 64.5) (end 377.772792 64.5) (width 0.25) (layer "B.Cu") (net 82))
+  (segment (start 360.4 68.8) (end 360.4 68.9) (width 0.25) (layer "B.Cu") (net 82))
   (segment (start 360.4 91.9375) (end 359.6275 92.71) (width 0.25) (layer "B.Cu") (net 82))
-  (segment (start 349.7 63.6) (end 352.5 63.6) (width 0.25) (layer "B.Cu") (net 82))
+  (segment (start 358.3 66.7) (end 360.4 68.8) (width 0.25) (layer "B.Cu") (net 82))
   (segment (start 369.8 75.8) (end 361 75.8) (width 0.25) (layer "B.Cu") (net 82))
   (segment (start 374.55 75.15) (end 374.55 66.495228) (width 0.25) (layer "B.Cu") (net 82))
@@
   (segment (start 379.746396 64.05) (end 380.196396 63.6) (width 0.25) (layer "B.Cu") (net 82))
   (segment (start 373.9 75.8) (end 374.55 75.15) (width 0.25) (layer "B.Cu") (net 82))
+  (segment (start 354.9 63.3) (end 354.9 65.3) (width 0.25) (layer "B.Cu") (net 82))
+  (segment (start 353.9 62.3) (end 354.9 63.3) (width 0.25) (layer "B.Cu") (net 82))
   (segment (start 378.222792 64.05) (end 379.746396 64.05) (width 0.25) (layer "B.Cu") (net 82))
-  (segment (start 352.5 63.6) (end 360.4 71.5) (width 0.25) (layer "B.Cu") (net 82))
+  (segment (start 348.4 62.3) (end 353.9 62.3) (width 0.25) (layer "B.Cu") (net 82))
   (segment (start 374.55 66.495228) (end 376.545228 64.5) (width 0.25) (layer "B.Cu") (net 82))
-  (segment (start 345.34 59.24) (end 349.7 63.6) (width 0.25) (layer "B.Cu") (net 82))
-  (segment (start 345.34 49.8475) (end 345.34 59.24) (width 0.25) (layer "B.Cu") (net 82))
   (segment (start 361 75.8) (end 360.4 76.4) (width 0.25) (layer "B.Cu") (net 82))
-  (segment (start 364.9 67) (end 360.4 71.5) (width 0.25) (layer "B.Cu") (net 82))
   (segment (start 364.2725 54.9275) (end 364.2725 57.3725) (width 0.25) (layer "B.Cu") (net 82))
   (segment (start 364.2725 57.3725) (end 364.9 58) (width 0.25) (layer "B.Cu") (net 82))
+  (segment (start 345.34 49.8475) (end 345.34 59.24) (width 0.25) (layer "B.Cu") (net 82))
   (segment (start 378.6775 109.6775) (end 378.6775 111.76) (width 0.25) (layer "B.Cu") (net 82))
   (segment (start 380.196396 63.6) (end 382.536396 63.6) (width 0.25) (layer "B.Cu") (net 82))
+  (segment (start 345.34 59.24) (end 348.4 62.3) (width 0.25) (layer "B.Cu") (net 82))
   (segment (start 369.8 75.8) (end 373.9 75.8) (width 0.25) (layer "B.Cu") (net 82))
   (segment (start 383.04 63.096396) (end 383.04 61.46) (width 0.25) (layer "B.Cu") (net 82))
   (segment (start 360.4 71.5) (end 360.4 91.9375) (width 0.25) (layer "B.Cu") (net 82))
+  (segment (start 356.3 66.7) (end 358.3 66.7) (width 0.25) (layer "B.Cu") (net 82))
   (segment (start 377.772792 64.5) (end 378.222792 64.05) (width 0.25) (layer "B.Cu") (net 82))
+  (segment (start 354.9 65.3) (end 356.3 66.7) (width 0.25) (layer "B.Cu") (net 82))
   (zone (net 80) (net_name "GND") (layer "F.Cu") (hatch edge 0.5)
     (connect_pads (clearance 0.5))
