File: KiCad/KeeBar_MiddlePlate/KeeBar_MiddlePlate.kicad_pcb (KiCad board)
At the start: 2 copper layers, 376 x 86.5 mm, 79 parts, among them M2_1 Val**, M2_2 Val**, M2_3 Val**, M2_4 Val**, M2_5 Val**, M2_6 Val**, M2_7 Val**, M2_8 Val**, M2_9 Val**, SW1 SW_Push, SW10 SW_Push, SW11 SW_Push, SW12 SW_Push, SW13 SW_Push, SW14 SW_Push, SW15 SW_Push, SW16 SW_Push, SW17 SW_Push, SW18 SW_Push, SW19 SW_Push, SW2 SW_Push, SW20 SW_Push, SW21 SW_Push, SW22 SW_Push, SW23 SW_Push, SW24 SW_Push, SW25 SW_Push, SW26 SW_Push, SW27 SW_Push, SW28 SW_Push, SW29 SW_Push, SW3 SW_Push, SW30 SW_Push, SW31 SW_Push, SW32 SW_Push, SW33 SW_Push, SW34 SW_Push, SW35 SW_Push, SW36 SW_Push, SW37 SW_Push, SW38 SW_Push, SW39 SW_Push, SW4 SW_Push, SW40 SW_Push, SW41 SW_Push, SW42 SW_Push, SW43 SW_Push, SW44 SW_Push, SW45 SW_Push, SW46 SW_Push, SW47 SW_Push, SW48 SW_Push, SW49 SW_Push, SW5 SW_Push, SW50 SW_Push, SW51 SW_Push, SW52 SW_Push, SW53 SW_Push, SW54 SW_Push, SW55 SW_Push, SW56 SW_Push, SW57 SW_Push, SW58 SW_Push, SW59 SW_Push, SW6 SW_Push, SW60 SW_Push, SW7 SW_Push, SW8 SW_Push, SW9 SW_Push

Commit message: PCBフォーム用KiCADデータ
Parts:
- removed REF**: Stabilizer_Cherry_MX_7.00u, Mounting_Keyboard_Stabilizer:Stabilizer_Cherry_MX_7.00u
- removed REF** (x5): Stabilizer_Cherry_MX_2.00u, Mounting_Keyboard_Stabilizer:Stabilizer_Cherry_MX_2.00u
- removed REF** (x3): Stabilizer_Cherry_MX_3.00u, Mounting_Keyboard_Stabilizer:Stabilizer_Cherry_MX_3.00u
- removed REF**: Stabilizer_Cherry_MX_6.25u, Mounting_Keyboard_Stabilizer:Stabilizer_Cherry_MX_6.25u
- added D1: 1N4148W, foam:foam-cutout-diode, B.Cu at (38.1, 58.5)
- added D10: 1N4148W, foam:foam-cutout-diode, B.Cu at (233.4, 58.6)
- added D11: 1N4148W, foam:foam-cutout-diode, B.Cu at (252.4, 58.6)
- added D12: 1N4148W, foam:foam-cutout-diode, B.Cu at (271.5, 58.6)
- added D13: 1N4148W, foam:foam-cutout-diode, B.Cu at (290.5, 58.6)
- added D14: 1N4148W, foam:foam-cutout-diode, B.Cu at (309.6, 58.6)
- added D15: 1N4148W, foam:foam-cutout-diode, B.Cu at (338.2, 60.9)
- added D16: 1N4148W, foam:foam-cutout-diode, B.Cu at (352.4, 60.9)
- added D17: 1N4148W, foam:foam-cutout-diode, B.Cu at (40.5, 77.6)
- added D18: 1N4148W, foam:foam-cutout-diode, B.Cu at (66.7, 77.6)
- added D19: 1N4148W, foam:foam-cutout-diode, B.Cu at (85.7, 77.6)
- added D2: 1N4148W, foam:foam-cutout-diode, B.Cu at (61.9, 58.6)
- added D20: 1N4148W, foam:foam-cutout-diode, B.Cu at (104.8, 77.6)
- added D21: 1N4148W, foam:foam-cutout-diode, B.Cu at (123.8, 77.6)
- added D22: 1N4148W, foam:foam-cutout-diode, B.Cu at (142.9, 77.6)
- added D23: 1N4148W, foam:foam-cutout-diode, B.Cu at (171.4, 77.6)
- added D24: 1N4148W, foam:foam-cutout-diode, B.Cu at (190.5, 77.6)
- added D25: 1N4148W, foam:foam-cutout-diode, B.Cu at (209.6, 77.6)
- added D26: 1N4148W, foam:foam-cutout-diode, B.Cu at (238.1, 77.6)
- added D27: 1N4148W, foam:foam-cutout-diode, B.Cu at (257.2, 77.6)
- added D28: 1N4148W, foam:foam-cutout-diode, B.Cu at (276.2, 77.6)
- added D29: 1N4148W, foam:foam-cutout-diode, B.Cu at (295.3, 77.6)
- added D3: 1N4148W, foam:foam-cutout-diode, B.Cu at (81.0, 58.6)
- added D30: 1N4148W, foam:foam-cutout-diode, B.Cu at (314.3, 77.6)
- added D31: 1N4148W, foam:foam-cutout-diode, B.Cu at (345.3, 77.6)
- added D32: 1N4148W, foam:foam-cutout-diode, B.Cu at (42.9, 96.7)
- added D33: 1N4148W, foam:foam-cutout-diode, B.Cu at (71.4, 96.7)
- added D34: 1N4148W, foam:foam-cutout-diode, B.Cu at (90.5, 96.7)
- added D35: 1N4148W, foam:foam-cutout-diode, B.Cu at (109.5, 96.7)
- added D36: 1N4148W, foam:foam-cutout-diode, B.Cu at (128.6, 96.7)
- added D37: 1N4148W, foam:foam-cutout-diode, B.Cu at (147.6, 96.7)
- added D38: 1N4148W, foam:foam-cutout-diode, B.Cu at (176.2, 96.7)
- added D39: 1N4148W, foam:foam-cutout-diode, B.Cu at (195.3, 96.7)
- added D4: 1N4148W, foam:foam-cutout-diode, B.Cu at (100.0, 58.6)
- added D40: 1N4148W, foam:foam-cutout-diode, B.Cu at (214.3, 96.7)
- added D41: 1N4148W, foam:foam-cutout-diode, B.Cu at (242.9, 96.7)
- added D42: 1N4148W, foam:foam-cutout-diode, B.Cu at (261.9, 96.7)
- added D43: 1N4148W, foam:foam-cutout-diode, B.Cu at (281.0, 96.7)
- added D44: 1N4148W, foam:foam-cutout-diode, B.Cu at (300.0, 96.7)
- added D45: 1N4148W, foam:foam-cutout-diode, B.Cu at (319.1, 96.7)
- added D46: 1N4148W, foam:foam-cutout-diode, B.Cu at (340.5, 96.7)
- added D47: 1N4148W, foam:foam-cutout-diode, B.Cu at (366.7, 101.4)
- added D48: 1N4148W, foam:foam-cutout-diode, B.Cu at (38.1, 115.7)
- added D49: 1N4148W, foam:foam-cutout-diode, B.Cu at (61.9, 115.7)
- added D5: 1N4148W, foam:foam-cutout-diode, B.Cu at (119.1, 58.6)
- added D50: 1N4148W, foam:foam-cutout-diode, B.Cu at (83.3, 115.7)
- added D51: 1N4148W, foam:foam-cutout-diode, B.Cu at (107.2, 115.7)
- added D52: 1N4148W, foam:foam-cutout-diode, B.Cu at (150.0, 109.5)
- added D53: 1N4148W, foam:foam-cutout-diode, B.Cu at (178.6, 119.1)
- added D54: 1N4148W, foam:foam-cutout-diode, B.Cu at (235.7, 109.5)
- added D55: 1N4148W, foam:foam-cutout-diode, B.Cu at (273.8, 115.7)
- added D56: 1N4148W, foam:foam-cutout-diode, B.Cu at (297.7, 115.7)
- added D57: 1N4148W, foam:foam-cutout-diode, B.Cu at (321.5, 115.7)
- added D58: 1N4148W, foam:foam-cutout-diode, B.Cu at (347.7, 119.5)
- added D59: 1N4148W, foam:foam-cutout-diode, B.Cu at (366.7, 119.5)
- added D6: 1N4148W, foam:foam-cutout-diode, B.Cu at (138.1, 58.6)
- added D60: 1N4148W, foam:foam-cutout-diode, B.Cu at (385.8, 119.5)
- added D7: 1N4148W, foam:foam-cutout-diode, B.Cu at (166.7, 58.6)
- added D8: 1N4148W, foam:foam-cutout-diode, B.Cu at (185.7, 58.6)
- added D9: 1N4148W, foam:foam-cutout-diode, B.Cu at (204.8, 58.6)
- added SW15-2: SW_Push, foam:foam-cutout-mx-socket, F.Cu at (333.4, 52.4)
- added SW16-2: SW_Push, foam:foam-cutout-mx-socket, F.Cu at (357.2, 52.4)
- added SW53-2: SW_Push, foam:foam-cutout-mx-socket, F.Cu at (195.3, 114.3)
- M2_1, M2_2, M2_3, M2_4, M2_5, M2_6, M2_7, M2_8, M2_9: footprint kbd_Hole:m2_Spacer_Hole_EdgeCuts -> foam:foam-cutout-hole-for-m2-hex
- SW1, SW10, SW11, SW12, SW13, SW14, SW15, SW16, SW17, SW18, SW19, SW2, SW20, SW21, SW22, SW23, SW24, SW25, SW26, SW27, SW28, SW29, SW3, SW30, SW31, SW32, SW33, SW34, SW35, SW36, SW37, SW38, SW39, SW4, SW40, SW41, SW42, SW43, SW44, SW45, SW46, SW47, SW48, SW49, SW5, SW50, SW51, SW52, SW53, SW54, SW55, SW56, SW57, SW58, SW59, SW6, SW60, SW7, SW8, SW9: footprint KeeBar:Swithch_hole_for_form -> foam:foam-cutout-mx-socket
- moved M2_3 25.0 mm to (287.0, 62.0)
- moved M2_8 23.7 mm to (287.0, 104.8)
- moved M2_4 16.2 mm to (361.5, 62.0)
- moved M2_9 12.2 mm to (361.5, 104.8)
- moved M2_5 5.83 mm to (205.0, 83.5)
- moved SW54 4.76 mm to (235.7, 114.3), turned to 180 degrees
- moved SW15 4.76 mm to (328.6, 52.4)
- moved SW16 4.76 mm to (352.4, 52.4)
- moved M2_7 3.34 mm to (117.0, 104.8)
- moved M2_1 2.50 mm to (50.0, 62.0)
- moved M2_2 2.50 mm to (117.0, 62.0)
- moved M2_6 2.30 mm to (50.0, 104.8)
- turned SW52 to 180 degrees
Other:
- outline, holes or cut-outs redrawn
- board text removed: "KeeBar v1.0 @ymkn"

Commit message: スタビ用の穴をあけ忘れていたのを修正
Parts:
- added ?: foam-cutout-mx-stab-2u, foam:foam-cutout-mx-stab-2u, F.Cu at (345.3, 71.4)
- added ?: foam-cutout-mx-stab-2u, foam:foam-cutout-mx-stab-2u, F.Cu at (235.7, 114.3)
- added ?: foam-cutout-mx-stab-6.25u, foam:foam-cutout-mx-stab-6.25u, F.Cu at (190.5, 114.3)
- added ?: foam-cutout-mx-stab-7u, foam:foam-cutout-mx-stab-7u, F.Cu at (190.5, 114.3)
- added ?: foam-cutout-mx-stab-2u, foam:foam-cutout-mx-stab-2u, F.Cu at (42.9, 90.5)
- added ?: foam-cutout-mx-stab-2u, foam:foam-cutout-mx-stab-2u, F.Cu at (195.3, 114.3)
- added ?: foam-cutout-mx-stab-2u, foam:foam-cutout-mx-stab-2u, F.Cu at (150.0, 114.3)
Changed lines of the file:
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@@
+      (stroke (width 0.05) (type default)) (fill none) (layer "Edge.Cuts"))
+  )
+  (footprint "foam:foam-cutout-mx-stab-2u" (layer "F.Cu")
+    (at 345.28125 71.4375)
+    (attr smd)
+    (fp_text reference "" (at 0.012 -0.485 unlocked) (layer "F.SilkS") hide
+        (effects (font (size 1 1) (thickness 0.1)))
+    )
+    (fp_text value "foam-cutout-mx-stab-2u" (at 0.012 1.015 unlocked) (layer "F.Fab") hide
+        (effects (font (size 1 1) (thickness 0.15)))
+    )
+    (fp_text user "${REFERENCE}" (at 0 0) (layer "F.Fab")
+        (effects (font (size 1 1) (thickness 0.15)))
+    )
+    (fp_circle (center -11.938 -6.985) (end -10.388 -6.985)
+      (stroke (width 0.1) (type default)) (fill none) (layer "Edge.Cuts"))
+    (fp_circle (center -11.938 8.225) (end -9.938 8.225)
+      (stroke (width 0.05) (type default)) (fill none) (layer "Edge.Cuts"))
+    (fp_circle (center 11.938 -6.985) (end 13.488 -6.985)
+      (stroke (width 0.1) (type default)) (fill none) (layer "Edge.Cuts"))
+    (fp_circle (center 11.938 8.225) (end 13.938 8.225)
       (stroke (width 0.05) (type default)) (fill none) (layer "Edge.Cuts"))
   )
@@
       (stroke (width 0.05) (type default)) (fill none) (layer "Edge.Cuts"))
   )
+  (footprint "foam:foam-cutout-mx-stab-2u" (layer "F.Cu")
+    (at 235.74375 114.3 180)
+    (attr smd)
+    (fp_text reference "" (at 0.012 -0.485 180 unlocked) (layer "F.SilkS") hide
+        (effects (font (size 1 1) (thickness 0.1)))
+    )
+    (fp_text value "foam-cutout-mx-stab-2u" (at 0.012 1.015 180 unlocked) (layer "F.Fab") hide
+        (effects (font (size 1 1) (thickness 0.15)))
+    )
+    (fp_circle (center -11.938 -6.985) (end -10.388 -6.985)
+      (stroke (width 0.1) (type default)) (fill none) (layer "Edge.Cuts"))
+    (fp_circle (center -11.938 8.225) (end -9.938 8.225)
+      (stroke (width 0.05) (type default)) (fill none) (layer "Edge.Cuts"))
+    (fp_circle (center 11.938 -6.985) (end 13.488 -6.985)
+      (stroke (width 0.1) (type default)) (fill none) (layer "Edge.Cuts"))
+    (fp_circle (center 11.938 8.225) (end 13.938 8.225)
+      (stroke (width 0.05) (type default)) (fill none) (layer "Edge.Cuts"))
+  )
   (footprint "foam:foam-cutout-mx-socket" (layer "F.Cu")
     (at 90.4875 90.4875)
@@
       (stroke (width 0.05) (type default)) (fill none) (layer "Edge.Cuts"))
   )
+  (footprint "foam:foam-cutout-mx-stab-6.25u" (layer "F.Cu")
+    (at 190.5 114.3 180)
+    (attr smd)
+    (fp_text reference "" (at 0.012 -0.485 180 unlocked) (layer "F.SilkS") hide
+        (effects (font (size 1 1) (thickness 0.1)))
+    )
+    (fp_text value "foam-cutout-mx-stab-6.25u" (at 0.012 1.015 180 unlocked) (layer "F.Fab") hide
+        (effects (font (size 1 1) (thickness 0.15)))
+    )
+    (fp_text user "${REFERENCE}" (at 0 0) (layer "F.Fab")
+        (effects (font (size 1 1) (thickness 0.15)))
+    )
+    (fp_circle (center -50 -6.985) (end -48.45 -6.985)
+      (stroke (width 0.1) (type default)) (fill none) (layer "Edge.Cuts"))
+    (fp_circle (center -50 8.225) (end -48 8.225)
+      (stroke (width 0.05) (type default)) (fill none) (layer "Edge.Cuts"))
+    (fp_circle (center 50 -6.985) (end 51.55 -6.985)
+      (stroke (width 0.1) (type default)) (fill none) (layer "Edge.Cuts"))
+    (fp_circle (center 50 8.225) (end 52 8.225)
+      (stroke (width 0.05) (type default)) (fill none) (layer "Edge.Cuts"))
+  )
   (footprint "foam:foam-cutout-mx-socket" (layer "F.Cu")
     (at 195.2625 90.4875)
@@
       (stroke (width 0.05) (type default)) (fill none) (layer "Edge.Cuts"))
   )
+  (footprint "foam:foam-cutout-mx-stab-7u" (layer "F.Cu")
+    (at 190.5 114.3 180)
+    (attr smd)
+    (fp_text reference "" (at 0.012 -0.485 180 unlocked) (layer "F.SilkS") hide
+        (effects (font (size 1 1) (thickness 0.1)))
+    )
+    (fp_text value "foam-cutout-mx-stab-7u" (at 0.012 1.015 180 unlocked) (layer "F.Fab") hide
+        (effects (font (size 1 1) (thickness 0.15)))
+    )
+    (fp_text user "${REFERENCE}" (at 0 0) (layer "F.Fab")
+        (effects (font (size 1 1) (thickness 0.15)))
+    )
+    (fp_circle (center -57.15 -6.985) (end -55.6 -6.985)
+      (stroke (width 0.1) (type default)) (fill none) (layer "Edge.Cuts"))
+    (fp_circle (center -57.15 8.225) (end -55.15 8.225)
+      (stroke (width 0.05) (type default)) (fill none) (layer "Edge.Cuts"))
+    (fp_circle (center 57.15 -6.985) (end 58.7 -6.985)
+      (stroke (width 0.1) (type default)) (fill none) (layer "Edge.Cuts"))
+    (fp_circle (center 57.15 8.225) (end 59.15 8.225)
+      (stroke (width 0.05) (type default)) (fill none) (layer "Edge.Cuts"))
+  )
   (footprint "foam:foam-cutout-mx-socket" (layer "F.Cu")
     (at 328.6125 52.3875)
@@
       (stroke (width 0.05) (type default)) (fill none) (layer "Edge.Cuts"))
   )
+  (footprint "foam:foam-cutout-mx-stab-2u" (layer "F.Cu")
+    (at 42.8625 90.4875)
+    (attr smd)
+    (fp_text reference "" (at 0.012 -0.485 unlocked) (layer "F.SilkS") hide
+        (effects (font (size 1 1) (thickness 0.1)))
+    )
+    (fp_text value "foam-cutout-mx-stab-2u" (at 0.012 1.015 unlocked) (layer "F.Fab") hide
+        (effects (font (size 1 1) (thickness 0.15)))
+    )
+    (fp_circle (center -11.938 -6.985) (end -10.388 -6.985)
+      (stroke (width 0.1) (type default)) (fill none) (layer "Edge.Cuts"))
+    (fp_circle (center -11.938 8.225) (end -9.938 8.225)
+      (stroke (width 0.05) (type default)) (fill none) (layer "Edge.Cuts"))
+    (fp_circle (center 11.938 -6.985) (end 13.488 -6.985)
+      (stroke (width 0.1) (type default)) (fill none) (layer "Edge.Cuts"))
+    (fp_circle (center 11.938 8.225) (end 13.938 8.225)
+      (stroke (width 0.05) (type default)) (fill none) (layer "Edge.Cuts"))
+  )
   (footprint "foam:foam-cutout-mx-socket" (layer "F.Cu")
     (at 71.4375 90.4875)
@@
       (stroke (width 0.05) (type default)) (fill none) (layer "Edge.Cuts"))
   )
+  (footprint "foam:foam-cutout-mx-stab-2u" (layer "F.Cu")
+    (at 195.2625 114.3 180)
+    (attr smd)
+    (fp_text reference "" (at 0.012 -0.485 180 unlocked) (layer "F.SilkS") hide
+        (effects (font (size 1 1) (thickness 0.1)))
+    )
+    (fp_text value "foam-cutout-mx-stab-2u" (at 0.012 1.015 180 unlocked) (layer "F.Fab") hide
+        (effects (font (size 1 1) (thickness 0.15)))
+    )
+    (fp_circle (center -11.938 -6.985) (end -10.388 -6.985)
+      (stroke (width 0.1) (type default)) (fill none) (layer "Edge.Cuts"))
+    (fp_circle (center -11.938 8.225) (end -9.938 8.225)
+      (stroke (width 0.05) (type default)) (fill none) (layer "Edge.Cuts"))
+    (fp_circle (center 11.938 -6.985) (end 13.488 -6.985)
+      (stroke (width 0.1) (type default)) (fill none) (layer "Edge.Cuts"))
+    (fp_circle (center 11.938 8.225) (end 13.938 8.225)
+      (stroke (width 0.05) (type default)) (fill none) (layer "Edge.Cuts"))
+  )
+  (footprint "foam:foam-cutout-mx-stab-2u" (layer "F.Cu")
+    (at 150.01875 114.3 180)
+    (attr smd)
+    (fp_text reference "" (at 0.012 -0.485 180 unlocked) (layer "F.SilkS") hide
+        (effects (font (size 1 1) (thickness 0.1)))
+    )
+    (fp_text value "foam-cutout-mx-stab-2u" (at 0.012 1.015 180 unlocked) (layer "F.Fab") hide
+        (effects (font (size 1 1) (thickness 0.15)))
+    )
+    (fp_circle (center -11.938 -6.985) (end -10.388 -6.985)
+      (stroke (width 0.1) (type default)) (fill none) (layer "Edge.Cuts"))
+    (fp_circle (center -11.938 8.225) (end -9.938 8.225)
+      (stroke (width 0.05) (type default)) (fill none) (layer "Edge.Cuts"))
+    (fp_circle (center 11.938 -6.985) (end 13.488 -6.985)
+      (stroke (width 0.1) (type default)) (fill none) (layer "Edge.Cuts"))
+    (fp_circle (center 11.938 8.225) (end 13.938 8.225)
+      (stroke (width 0.05) (type default)) (fill none) (layer "Edge.Cuts"))
+  )
